File: VersiB/KICAD/ExpansionBoard-V2.0.kicad_pcb (KiCad board)
At the start: 2 copper layers, 101.6 x 53.3 mm, 83 parts, among them J1 Power, J10 Conn_01x04, J11 Conn_01x04, J12 Conn_01x04, J2 Analog, J3 Analog, J4 Digital, J5 PWM, J6 PWM, J7 Communication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

Commit message: update
Parts:
- R31: value 1K -> 100
