File: VersiB/KICAD/ExpansionBoard-V2.0.kicad_sch (KiCad schematic)
At the start: 76 parts, among them J1 Power, J10 Conn_01x04, J11 Conn_01x04, J12 Conn_01x04, J2 Analog, J3 Analog, J4 Digital, J5 PWM, J6 PWM, J7 Communication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

Commit message: update
Parts:
- R31: value 1K -> 100

Commit message: update
Other:
- moved on the sheet: R29
Changed lines of the file:
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@@
 	)
 	(junction
+		(at 261.62 44.45)
+		(diameter 0)
+		(color 0 0 0 0)
+	)
+	(junction
 		(at 102.87 60.96)
 		(diameter 0)
@@
 	)
 	(junction
-		(at 262.89 44.45)
-		(diameter 0)
-		(color 0 0 0 0)
-	)
-	(junction
 		(at 102.87 46.99)
 		(diameter 0)
@@
 	(wire
 		(pts
-			(xy 262.89 44.45) (xy 264.16 44.45)
-		)
-		(stroke
-			(width 0)
-			(type default)
-		)
-	)
-	(wire
-		(pts
 			(xy 78.74 43.18) (xy 78.74 45.72)
 		)
@@
 	(wire
 		(pts
-			(xy 262.89 54.61) (xy 262.89 57.15)
+			(xy 261.62 54.61) (xy 261.62 55.88)
 		)
 		(stroke
@@
 	(wire
 		(pts
-			(xy 250.19 44.45) (xy 262.89 44.45)
+			(xy 250.19 44.45) (xy 261.62 44.45)
 		)
 		(stroke
@@
 	(wire
 		(pts
-			(xy 262.89 44.45) (xy 262.89 46.99)
+			(xy 261.62 44.45) (xy 261.62 46.99)
 		)
 		(stroke
@@
 	(wire
 		(pts
+			(xy 261.62 55.88) (xy 262.89 55.88)
+		)
+		(stroke
+			(width 0)
+			(type default)
+		)
+	)
+	(wire
+		(pts
 			(xy 238.76 34.29) (xy 238.76 35.56)
 		)
@@
 	(wire
 		(pts
+			(xy 262.89 55.88) (xy 262.89 57.15)
+		)
+		(stroke
+			(width 0)
+			(type default)
+		)
+	)
+	(wire
+		(pts
 			(xy 44.45 109.22) (xy 44.45 119.38)
 		)
@@
 	(wire
 		(pts
+			(xy 261.62 44.45) (xy 264.16 44.45)
+		)
+		(stroke
+			(width 0)
+			(type default)
+		)
+	)
+	(wire
+		(pts
 			(xy 154.94 33.02) (xy 154.94 35.56)
 		)
@@
 	(symbol
 		(lib_id "Device:R")
-		(at 262.89 50.8 0)
+		(at 261.62 50.8 0)
 		(unit 1)
 		(body_style 1)
@@
 		(fields_autoplaced yes)
 		(property "Reference" "R29"
-			(at 265.43 49.5299 0)
+			(at 264.16 49.5299 0)
 			(show_name no)
 			(do_not_autoplace no)
@@
 		)
 		(property "Value" "1M"
-			(at 265.43 52.0699 0)
+			(at 264.16 52.0699 0)
 			(show_name no)
 			(do_not_autoplace no)
@@
 		)
 		(property "Footprint" "Resistor_SMD:R_0805_2012Metric_Pad1.20x1.40mm_HandSolder"
-			(at 261.112 50.8 90)
+			(at 259.842 50.8 90)
 			(hide yes)
 			(show_name no)
@@
 		)
 		(property "Datasheet" ""
-			(at 262.89 50.8 0)
+			(at 261.62 50.8 0)
 			(hide yes)
 			(show_name no)
@@
 		)
 		(property "Description" "Resistor"
-			(at 262.89 50.8 0)
+			(at 261.62 50.8 0)
 			(hide yes)
 			(show_name no)
