File: versiA/Kicad/ExpansionBoard-V2.0.kicad_pcb (KiCad board)
At the start: 2 copper layers, 101.6 x 53.3 mm, 84 parts, among them J1 Power, J10 Conn_01x04, J11 Conn_01x04, J12 Conn_01x04, J2 Analog, J3 Analog, J4 Digital, J5 PWM, J6 PWM, J7 Communication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

Commit message: update
Parts:
- R31: value 1K -> 100
Changed lines of the file:
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@@
 		(sheetname "/")
 		(sheetfile "ExpansionBoard-V2.0.kicad_sch")
+		(units
+			(unit
+				(name "A")
+				(pins "1" "3" "5" "7" "9" "11" "13" "15" "17" "19" "21" "23" "25" "27"
+					"29" "31" "33" "35" "2" "4" "6" "8" "10" "12" "14" "16" "18" "20" "22"
+					"24" "26" "28" "30" "32" "34" "36"
+				)
+			)
+		)
 		(attr through_hole)
 		(duplicate_pad_numbers_are_jumpers no)
@@
 		(sheetname "/")
 		(sheetfile "ExpansionBoard-V2.0.kicad_sch")
+		(units
+			(unit
+				(name "A")
+				(pins "1" "2" "3" "4" "5" "6" "7" "8")
+			)
+		)
 		(attr through_hole)
 		(duplicate_pad_numbers_are_jumpers no)
@@
 		(sheetname "/")
 		(sheetfile "ExpansionBoard-V2.0.kicad_sch")
+		(units
+			(unit
+				(name "A")
+				(pins "1" "2" "3" "4" "5" "6" "7" "8")
+			)
+		)
 		(attr through_hole)
 		(duplicate_pad_numbers_are_jumpers no)
@@
 		(sheetname "/")
 		(sheetfile "ExpansionBoard-V2.0.kicad_sch")
+		(units
+			(unit
+				(name "A")
+				(pins "1" "2" "3" "4" "5" "6" "7" "8")
+			)
+		)
 		(attr through_hole)
 		(duplicate_pad_numbers_are_jumpers no)
@@
 		(sheetname "/")
 		(sheetfile "ExpansionBoard-V2.0.kicad_sch")
+		(units
+			(unit
+				(name "A")
+				(pins "1" "2" "3" "4" "5" "6" "7" "8" "9" "10")
+			)
+		)
 		(attr through_hole)
 		(duplicate_pad_numbers_are_jumpers no)
@@
 		(sheetname "/")
 		(sheetfile "ExpansionBoard-V2.0.kicad_sch")
+		(units
+			(unit
+				(name "A")
+				(pins "1" "2" "3" "4" "5" "6" "7" "8")
+			)
+		)
 		(attr through_hole)
 		(duplicate_pad_numbers_are_jumpers no)
@@
 		(sheetname "/")
 		(sheetfile "ExpansionBoard-V2.0.kicad_sch")
+		(units
+			(unit
+				(name "A")
+				(pins "1" "2" "3" "4" "5" "6" "7" "8")
+			)
+		)
 		(attr through_hole)
 		(duplicate_pad_numbers_are_jumpers no)
@@
 			)
 		)
-		(property "Value" "1K"
+		(property "Value" "100"
 			(at -0.15 2.12 0)
 			(layer "F.Fab")
