File: versiA/Kicad/ExpansionBoard-V2.0.kicad_sch (KiCad schematic)
At the start: 76 parts, among them J1 Power, J10 Conn_01x04, J11 Conn_01x04, J12 Conn_01x04, J2 Analog, J3 Analog, J4 Digital, J5 PWM, J6 PWM, J7 Communication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

Commit message: update
Parts:
- R31: value 1K -> 100
Changed lines of the file:
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@@
 			)
 		)
-		(property "Value" "1K"
+		(property "Value" "100"
 			(at 274.32 35.5599 0)
 			(show_name no)
